Commit message: asdfas

File: basic134/urdf/threedofexample.urdf (robot description, URDF)
Before this commit: robot threedofexample, 9 links, 8 joints
Links:
- removed link tip
- added link endbracket; visual mesh filename=package://basic134/meshes/wrist.STL scale=0.001 0.001 0.001
- added link final
- added link final2; visual mesh filename=package://basic134/meshes/end_effector_v2.STL scale=0.001 0.001 0.001
- added link wristmotor; visual mesh filename=package://basic134/meshes/X5.stl scale=0.001 0.001 0.001
- link basemotor: geometry visual mesh filename=package://basic134/meshes/X8.stl scale=0.001 0.001 0.001
- link baseplate: geometry visual mesh filename=package://basic134/meshes/base.STL scale=0.001 0.001 0.001
- link lbracket: geometry visual mesh filename=package://basic134/meshes/shoulder.STL scale=0.001 0.001 0.001
- link lowerarm: geometry visual mesh filename=package://basic134/meshes/second_link.STL scale=0.001 0.001 0.001
- link upperarm: geometry visual mesh filename=package://basic134/meshes/first_link.STL scale=0.001 0.001 0.001
Joints:
- added joint endmotor: type fixed, parent endbracket, child final, origin xyz=0 0 0 rpy=0 0 0
- added joint final: type continuous, parent final, child final2, origin xyz=0.0 0.041 -0.03 rpy=0 0 0, axis 0 0 1
- added joint wrist: type continuous, parent wristmotor, child endbracket, origin xyz=0 0.0516 0 rpy=0 0 0, axis 0 1 0
- joint base: origin xyz=0 0 0.04185 rpy=0 0 3.1459 -> xyz=0 0 0.0451 rpy=0 0 0
- joint elbow: axis 0 0 1 -> 0 1 0; origin xyz=0 0 0.0311 rpy=0 0 3.1459 -> xyz=0 -0.0376 0 rpy=0 0 0
- joint lbracket: origin xyz=0 -0.0311 0.05 rpy=-1.5708 1.5708 0 -> xyz=0 -0.0225 0.0575 rpy=0 0 0
- joint lowerarm: child tip -> wristmotor; origin xyz=-0.378 0 0 rpy=0 0 3.1459 -> xyz=0.647 0.0065 0.0035 rpy=0 0 0
- joint placement: origin xyz=-0.0585 0 0 rpy=0 0 0 -> xyz=0 0 0 rpy=0 0 0
- joint shoulder: axis 0 0 1 -> 0 1 0; origin xyz=0 0 0.04698 rpy=0 0 1.5708 -> xyz=0 0.0516 0 rpy=0 0 0
- joint upperarm: origin xyz=0.402 0 0.00572 rpy=0 0 0 -> xyz=0.445 -0.00635 0.004 rpy=0 0 0

Commit message: working bot

File: basic134/urdf/threedofexample.urdf (robot description, URDF)
Before this commit: robot threedofexample, 12 links, 11 joints
Links:
- removed link final
- removed link final2
- added link endmotor; visual mesh filename=package://basic134/meshes/end_effector_v2.STL scale=0.001 0.001 0.001
Joints:
- removed joint endmotor
- removed joint final
- added joint end: type continuous, parent endbracket, child endmotor, origin xyz=0.0 0.041 -0.03 rpy=0 0 0, axis 0 0 1
- joint elbow: axis 0 1 0 -> 0 -1 0

Commit message: aruco work

File: basic134/urdf/threedofexample.urdf (robot description, URDF)
Before this commit: robot threedofexample, 11 links, 10 joints
Joints:
- joint baseplate: origin xyz=-0.0215 0 0.0125 rpy=0 0 0 -> xyz=-0.0025 -0.002 0.0125 rpy=0 0 0
- joint lowerarm: origin xyz=0.647 0.0065 0.0035 rpy=0 0 0 -> xyz=0.647 0.0065 0.001 rpy=0 0 0
- joint placement: origin xyz=0 0 0 rpy=0 0 0 -> xyz=0.03387 0.08992 0 rpy=0 0 0
- joint upperarm: origin xyz=0.445 -0.00635 0.004 rpy=0 0 0 -> xyz=0.445 -0.00635 0.003 rpy=0 0 0

Commit message: asdf

File: basic134/urdf/threedofexample.urdf (robot description, URDF)
Before this commit: robot threedofexample, 11 links, 10 joints
Links:
- link lowerarm: geometry visual mesh filename=package://basic134/meshes/first_link.STL scale=0.001 0.001 0.001
Joints:
- joint lowerarm: origin xyz=0.647 0.0065 0.001 rpy=0 0 0 -> xyz=0.446 0.0075 0.001 rpy=0 0 0

Commit message: manip working

File: basic134/urdf/threedofexample.urdf (robot description, URDF)
Before this commit: robot threedofexample, 11 links, 10 joints
Joints:
- joint base: origin xyz=0 0 0.0451 rpy=0 0 0 -> xyz=0 0 0.041 rpy=0 0 0
- joint elbow: origin xyz=0 -0.0376 0 rpy=0 0 0 -> xyz=0 -0.0384 0 rpy=0 0 0
- joint end: axis 0 0 1 -> 0 0 -1
- joint lbracket: origin xyz=0 -0.0225 0.0575 rpy=0 0 0 -> xyz=0 -0.025 0.069 rpy=0 0 0
